File: hardware/v2/fan.kicad_sch (KiCad schematic)
At the start: 25 parts, among them J301 B3P-VH-B, J302 B5B-XH-A, U301 MCT8315Z0HRRYR

Commit message: Complete draft of the v2 PCB
Parts:
- RV301: Label (none) -> FAN CURRENT LIMIT
- TP301: footprint TestPoint:TestPoint_2Pads_Pitch5.08mm_Drill1.3mm -> TestPoint:TestPoint_2Pads_Pitch2.54mm_Drill0.8mm
Connections:
- net GND: now also U301.34 (EP), U301.35 (EP), U301.36 (EP), U301.37 (EP), U301.38 (EP), U301.39 (EP), U301.40 (EP), U301.41 (EP), U301.42 (EP), U301.43 (EP), U301.44 (EP)
Other:
- note added: "Increasing resistance of the setpoint increases the current limit"
- moved on the sheet: C306, R301, R302, R303, RV301, TP301

Commit message: Prepare Minuet v2 for fabrication.
Parts:
- R308: now left out of the parts list
Changed lines of the file:
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@@
 		(unit 1)
 		(exclude_from_sim no)
-		(in_bom yes)
+		(in_bom no)
 		(on_board yes)
 		(dnp yes)
