File: hardware/v2/minuet.kicad_sch (KiCad schematic)
At the start: 39 parts, among them J101 B2P-VH-B, J102 B2B-XH-A_1, J103 PPPC062LFBN-RC, J104 B2B-XH-A_1, Q101 MMBT3904, U101 TSOP39238, U102 LMV331X-SC5R

Commit message: Complete draft of the v2 PCB
Parts:
- removed NT103: NetTie_2, Generic:NetTie-2_SMD_Pad0.6mm, symbol Device:NetTie_2
- C101: value 680u -> 1000u; Part EKZH250ELL681MJ16S -> EKYB250ELL102MJ20S
- J102, J104: value B2B-XH-A_1 -> B2B-XH-A
- NT101: footprint Generic:NetTie-2_SMD_Pad0.6mm -> Generic:NetTie-2_SMD_Pad1.0mm
- NT102: footprint Generic:NetTie-2_SMD_Pad0.3mm -> Generic:NetTie-2_SMD_Pad0.2mm
- TP101, TP102: footprint TestPoint:TestPoint_Pad_1.5x1.5mm -> TestPoint:TestPoint_Pad_D1.0mm
- U102: footprint Package_TO_SOT_SMD:SOT-323_SC-70 -> Package_TO_SOT_SMD:SOT-353_SC-70-5
Connections:
- net +12V: no longer NT102.1
- net +3.3V: now also J103.10 (Pin_10), NT102.2; no longer J103.2 (Pin_2), VR101.7 (VOS)
- net BOOT: now also J103.1 (Pin_1); no longer J103.10 (Pin_10)
- net GND: now also J103.9 (Pin_9); no longer J103.1 (Pin_1)
- net GPIO0: now also J103.4 (Pin_4); no longer J103.3 (Pin_3)
- net GPIO1: now also J103.3 (Pin_3); no longer J103.4 (Pin_4)
- net GPIO3: now also C105.1, R103.1, R106.2; no longer J102.2 (Pin_2), R101.1
- net GPIO4: now also J102.2 (Pin_2), R101.1; no longer C105.1, R103.1, R106.2
- net RESET: now also J103.2 (Pin_2); no longer J103.9 (Pin_9)
- net SCL: now also J103.6 (Pin_6); no longer J103.7 (Pin_7)
- net SDA: now also J103.5 (Pin_5); no longer J103.8 (Pin_8)
- net UART_RXD: now also J103.7 (Pin_7); no longer J103.6 (Pin_6)
- net UART_TXD: now also J103.8 (Pin_8); no longer J103.5 (Pin_5)
- net XIO0: now also R115.1
- net XIO1: now also R116.1
- net XIO10: now also R113.2
- net XIO11: no longer R113.2
- net XIO13: now also R108.2
- net XIO14: no longer R101.2
- net XIO15: now also R101.2; no longer U102.4
- net XIO6: no longer R116.1
- net XIO7: no longer R115.1
- net XIO8: now also U102.4; no longer R108.2
- net 12V_PWR: now reaches JP101.3 (B)
- net 12V_PWR: now also C102.1, C103.1, NT101.2, R102.1, R103.2, VR101.1 (VIN)
- net RTHR: now reaches R109.1, R114.2, TP102.1, U102.3 (-)
- new net: NT102.1, VR101.7 (VOS)

Commit message: Prepare Minuet v2 for fabrication.
Parts:
- R101, R103, R106, R110: Rating (none) -> 1%
- R109: value 22K -> 100K; Rating (none) -> 1%
- R114: value 100K -> 1.5M
Connections:
- net RSEN: now reaches C106.1, R110.2, R111.2, TP101.1, U102.1 (+)
Other:
- note added: "Header for custom peripherals and factory programming - GPIO0 and GPIO1 are free to be used for any purpose - UART_RXD and UART_TXD provide the serial port - SCL and SDA provide the I2C bus (QWIIC) - RESET and BOOT are wired in parallel with their corresponding buttons (active when tied to ground) - 12 V supply is unregulated, 1 A maximum current - 3.3 V supply is regulated, 1 A maximum current"
- note added: "The rain sensor is only available on model 4500K; these components may be omitted for other models It is simply a pair of electrodes that are exposed to the environment and whose impedance is about 0.5 to 1.2 Mohm when in contact with water or mist and open circuit when dry The comparator pulls the output low when V(RSEN) < V(RTHR) + V(OFFSET), where V(OFFSET) is +/- 5 mV for LMV331X"
- note removed: "Header for custom peripherals and factory programming - GPIO0 and GPIO1 are free to be used for any purpose - UART_RXD and UART_TXD provide the serial port - SCL and SDA provide the I2C bus (QWIIC) - RESET and BOOT are wired in parallel with their corresponding buttons (active when tied to ground)"
- note removed: "The rain sensor is only available on model 4500K; these components may be omitted for other models It is simply a pair of electrodes that are exposed to the environment and whose impedance is about 0 to 300 Kohm when in contact with water and open circuit when dry"
- moved on the sheet: C106, J103
