File: hardware/light/light.kicad_pcb (KiCad board)
At the start: 2 copper layers, 25 x 30 mm, 18 parts, among them J1 PH2-12-UA, J2 Conn_01x07, J3 Conn_01x07, J4 B3B-XH-A, Q1 DMG2301L, Q2 MMBT3904, U1 LP2985-50DBVR, U2 SN74LVC1G17DBVR

Commit message: Finalize light accessory v2.5 for manufacture.
Parts:
- R3: value 1K -> 10K
Connections:
- C1 pad 1: +12V -> Net-(JP1-A)
Routing:
- net +12V: track 65.5 -> 59.6 mm
- net Net-(JP1-A): track 26.9 -> 31.5 mm
