File: hardware/light/light.kicad_sch (KiCad schematic)
At the start: 18 parts, among them J1 PH2-12-UA, J2 Conn_01x07, J3 Conn_01x07, J4 B3B-XH-A, Q1 DMG2301L, Q2 MMBT3904, U1 LP2985-50DBVR, U2 SN74LVC1G17DBVR

Commit message: Finalize light accessory v2.5 for manufacture.
Parts:
- C1: Rating 25V, X7R -> 25V, X5R
- C2: Rating X7R -> 25V, X5R
- C3: Rating 10V, X7R -> 6.3V, X5R
- R3: value 1K -> 10K
Connections:
- net +12V: no longer C1.1
- net at JP1.1 (A), U1.1 (VIN), U1.3 (ON/~{OFF}): now also C1.1
Other:
- note added: "Header for accessories and factory programming - GPIO0 and GPIO1 are free to be used for any purpose - UART_RXD and UART_TXD provide the serial port - SCL and SDA provide the I2C bus (QWIIC) - RESET and BOOT are wired in parallel with their corresponding buttons (active when tied to ground) - 12 V supply is unregulated, 1 A current available - 5 V supply is regulated, 150 mA current available - 3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"
- note added: "Supplies 150 mA, ultra low quiescent current (microamps)"
- note removed: "150 mA maximum current, ultra low quiescent current (microamps)"
- note removed: "Header for accessories and factory programming - GPIO0 and GPIO1 are free to be used for any purpose - UART_RXD and UART_TXD provide the serial port - SCL and SDA provide the I2C bus (QWIIC) - RESET and BOOT are wired in parallel with their corresponding buttons (active when tied to ground) - 12 V supply is unregulated, 1 A maximum current - 5 V supply is regulated, 150 mA maximum current - 3.3 V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"
- moved on the sheet: C1, JP1
Changed lines of the file:
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@@
 	)
 	(junction
-		(at 121.92 64.77)
-		(diameter 0)
-		(color 0 0 0 0)
-	)
-	(junction
 		(at 220.98 64.77)
 		(diameter 0)
@@
 	)
 	(junction
+		(at 130.81 67.31)
+		(diameter 0)
+		(color 0 0 0 0)
+	)
+	(junction
 		(at 220.98 101.6)
 		(diameter 0)
@@
 	(wire
 		(pts
-			(xy 121.92 64.77) (xy 121.92 69.85)
-		)
-		(stroke
-			(width 0)
-			(type default)
-		)
-	)
-	(wire
-		(pts
-			(xy 120.65 64.77) (xy 121.92 64.77)
+			(xy 119.38 64.77) (xy 120.65 64.77)
 		)
 		(stroke
@@
 	(wire
 		(pts
-			(xy 121.92 64.77) (xy 123.19 64.77)
+			(xy 128.27 116.84) (xy 133.35 116.84)
 		)
 		(stroke
@@
 	(wire
 		(pts
-			(xy 128.27 116.84) (xy 133.35 116.84)
+			(xy 220.98 74.93) (xy 227.33 74.93)
 		)
 		(stroke
@@
 	(wire
 		(pts
-			(xy 220.98 74.93) (xy 227.33 74.93)
+			(xy 66.04 96.52) (xy 63.5 96.52)
 		)
 		(stroke
@@
 	(wire
 		(pts
-			(xy 66.04 96.52) (xy 63.5 96.52)
+			(xy 157.48 116.84) (xy 160.02 116.84)
 		)
 		(stroke
@@
 	(wire
 		(pts
-			(xy 157.48 116.84) (xy 160.02 116.84)
+			(xy 133.35 116.84) (xy 133.35 118.11)
 		)
 		(stroke
@@
 	(wire
 		(pts
-			(xy 133.35 116.84) (xy 133.35 118.11)
+			(xy 81.28 128.27) (xy 83.82 128.27)
 		)
 		(stroke
@@
 	(wire
 		(pts
-			(xy 81.28 128.27) (xy 83.82 128.27)
+			(xy 234.95 82.55) (xy 237.49 82.55)
 		)
 		(stroke
@@
 	(wire
 		(pts
-			(xy 234.95 82.55) (xy 237.49 82.55)
+			(xy 130.81 67.31) (xy 130.81 69.85)
 		)
 		(stroke
@@
 	(wire
 		(pts
+			(xy 128.27 64.77) (xy 130.81 64.77)
+		)
+		(stroke
+			(width 0)
+			(type default)
+		)
+	)
+	(wire
+		(pts
 			(xy 81.28 115.57) (xy 83.82 115.57)
 		)
@@
 	(wire
 		(pts
-			(xy 121.92 81.28) (xy 142.24 81.28)
+			(xy 130.81 81.28) (xy 142.24 81.28)
 		)
 		(stroke
@@
 	(wire
 		(pts
-			(xy 121.92 77.47) (xy 121.92 81.28)
+			(xy 130.81 77.47) (xy 130.81 81.28)
 		)
 		(stroke
@@
 		)
 	)
-	(text "Header for accessories and factory programming\n- GPIO0 and GPIO1 are free to be used for any purpose\n- UART_RXD and UART_TXD provide the serial port\n- SCL and SDA provide the I2C bus (QWIIC)\n- RESET and BOOT are wired in parallel with their\n   corresponding buttons (active when tied to ground)\n- 12 V supply is unregulated, 1 A maximum current\n- 5 V supply is regulated, 150 mA maximum current\n- 3.3 V supply is regulated, 1 A maximum current"
+	(text "Header for accessories and factory programming\n- GPIO0 and GPIO1 are free to be used for any purpose\n- UART_RXD and UART_TXD provide the serial port\n- SCL and SDA provide the I2C bus (QWIIC)\n- RESET and BOOT are wired in parallel with their\n   corresponding buttons (active when tied to ground)\n- 12 V supply is unregulated, 1 A current available\n- 5 V supply is regulated, 150 mA current available\n- 3.3 V supply is regulated, 600 mA current available"
 		(exclude_from_sim no)
 		(at 41.91 54.61 0)
@@
 		)
 	)
-	(text "150 mA maximum current, ultra low quiescent current (microamps)"
+	(text "Supplies 150 mA, ultra low quiescent current (microamps)"
 		(exclude_from_sim no)
 		(at 109.22 54.61 0)
@@
 		(length 2.54)
 		(shape round)
-		(at 130.81 67.31 180)
+		(at 130.81 67.31 90)
 		(fields_autoplaced yes)
 		(effects
@@
 				(size 1.27 1.27)
 			)
-			(justify right bottom)
+			(justify left bottom)
 		)
 		(property "Netclass" "Power"
-			(at 131.5085 69.85 0)
+			(at 128.27 66.6115 90)
 			(effects
 				(font
@@
 			)
 		)
-		(property "Rating" "10V, X7R"
+		(property "Rating" "6.3V, X5R"
 			(at 174.371 77.2964 0)
 			(effects
@@
 	(symbol
 		(lib_id "power:+12V")
-		(at 120.65 64.77 90)
+		(at 119.38 64.77 90)
 		(unit 1)
 		(exclude_from_sim no)
@@
 		(fields_autoplaced yes)
 		(property "Reference" "#PWR02"
-			(at 124.46 64.77 0)
+			(at 123.19 64.77 0)
 			(effects
 				(font
@@
 		)
 		(property "Value" "+12V"
-			(at 117.475 64.77 90)
+			(at 116.205 64.77 90)
 			(effects
 				(font
@@
 		)
 		(property "Footprint" ""
-			(at 120.65 64.77 0)
+			(at 119.38 64.77 0)
 			(effects
 				(font
@@
 		)
 		(property "Datasheet" ""
-			(at 120.65 64.77 0)
+			(at 119.38 64.77 0)
 			(effects
 				(font
@@
 		)
 		(property "Description" "Power symbol creates a global label with name \"+12V\""
-			(at 120.65 64.77 0)
+			(at 119.38 64.77 0)
 			(effects
 				(font
@@
 	(symbol
 		(lib_id "Jumper:SolderJumper_2_Bridged")
-		(at 127 64.77 0)
-		(mirror y)
+		(at 124.46 64.77 180)
 		(unit 1)
 		(exclude_from_sim yes)
@@
 		(on_board yes)
 		(dnp no)
+		(fields_autoplaced yes)
 		(property "Reference" "JP1"
-			(at 127 67.3791 0)
+			(at 124.46 62.1609 0)
 			(effects
 				(font
@@
 		)
 		(property "Value" "SolderJumper_2_Open"
-			(at 128.2121 66.421 90)
+			(at 125.6721 63.119 90)
 			(effects
 				(font
@@
 		)
 		(property "Footprint" "Jumper:SolderJumper-2_P1.3mm_Bridged_RoundedPad1.0x1.5mm"
-			(at 127 64.77 0)
+			(at 124.46 64.77 0)
 			(effects
 				(font
@@
 		)
 		(property "Datasheet" "~"
-			(at 127 64.77 0)
+			(at 124.46 64.77 0)
 			(effects
 				(font
@@
 		)
 		(property "Description" "Solder Jumper, 2-pole, closed/bridged"
-			(at 127 64.77 0)
+			(at 124.46 64.77 0)
 			(effects
 				(font
@@
 		(on_board yes)
 		(dnp no)
-		(fields_autoplaced yes)
 		(property "Reference" "R4"
 			(at 210.3121 95.3078 0)
@@
 	(symbol
 		(lib_id "Device:C")
-		(at 121.92 73.66 0)
+		(at 130.81 73.66 0)
 		(mirror y)
 		(unit 1)
@@
 		(dnp no)
 		(property "Reference" "C1"
-			(at 118.999 70.0235 0)
+			(at 127.889 70.0235 0)
 			(effects
 				(font
@@
 		)
 		(property "Value" "1u"
-			(at 118.999 72.4478 0)
+			(at 127.889 72.4478 0)
 			(effects
 				(font
@@
 		)
 		(property "Footprint" "Capacitor_SMD:C_0603_1608Metric_Pad1.08x0.95mm_HandSolder"
-			(at 120.9548 77.47 0)
+			(at 129.8448 77.47 0)
 			(effects
 				(font
@@
 		)
 		(property "Datasheet" "~"
-			(at 121.92 73.66 0)
+			(at 130.81 73.66 0)
 			(effects
 				(font
@@
 		)
 		(property "Description" "Unpolarized capacitor"
-			(at 121.92 73.66 0)
+			(at 130.81 73.66 0)
 			(effects
 				(font
@@
 		)
 		(property "Arrow Part Number" ""
-			(at 121.92 73.66 0)
+			(at 130.81 73.66 0)
 			(effects
 				(font
@@
 		)
 		(property "Arrow Price/Stock" ""
-			(at 121.92 73.66 0)
+			(at 130.81 73.66 0)
 			(effects
 				(font
@@
 		)
 		(property "Height" ""
-			(at 121.92 73.66 0)
+			(at 130.81 73.66 0)
 			(effects
 				(font
@@
 		)
 		(property "Hold Current" ""
-			(at 121.92 73.66 0)
+			(at 130.81 73.66 0)
 			(effects
 				(font
@@
 		)
 		(property "Manufacturer_Name" ""
-			(at 121.92 73.66 0)
+			(at 130.81 73.66 0)
 			(effects
 				(font
@@
 		)
 		(property "Manufacturer_Part_Number" ""
-			(at 121.92 73.66 0)
+			(at 130.81 73.66 0)
 			(effects
 				(font
@@
 		)
 		(property "Mouser Part Number" ""
-			(at 121.92 73.66 0)
+			(at 130.81 73.66 0)
 			(effects
 				(font
@@
 		)
 		(property "Mouser Price/Stock" ""
-			(at 121.92 73.66 0)
+			(at 130.81 73.66 0)
 			(effects
 				(font
@@
 		)
 		(property "Type" "Ceramic"
-			(at 118.999 74.8721 0)
+			(at 127.889 74.8721 0)
 			(effects
 				(font
@@
 			)
 		)
-		(property "Rating" "25V, X7R"
-			(at 118.999 77.2964 0)
+		(property "Rating" "25V, X5R"
+			(at 127.889 77.2964 0)
 			(effects
 				(font
@@
 			)
 		)
-		(property "Rating" "X7R"
+		(property "Rating" "25V, X5R"
 			(at 159.131 77.2964 0)
 			(effects
@@
 			)
 		)
-		(property "Value" "1K"
+		(property "Value" "10K"
 			(at 207.01 88.7038 90)
 			(effects
