File: hardware/minuet/v2/core.kicad_sch (KiCad schematic)
At the start: 15 parts, among them J201 USB4105-GF-A, J202 SM04B-SRSS-TB, SW201 EVQ-P7A01P, SW202 EVQ-P7A01P, U201 TCA9555RTWR, U202 ESP32-C3-WROOM-02

Commit message: Wordsmithing accessories and components.
Other:
- note added: "Host has pull-ups so accessories don't need their own"
- note removed: "Host has pull-ups so peripherals don't need their own"
Changed lines of the file:
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@@
 		)
 	)
-	(text "Host has pull-ups so peripherals don't need their own"
+	(text "Host has pull-ups so accessories don't need their own"
 		(exclude_from_sim no)
 		(at 208.28 90.17 0)

Commit message: Finalize Minuet v2.1 for manufacture.
This revision uses a different motor controller and buck converter
and remedies errata from v2.0.
Parts:
- C201, C203, C204, C205: Rating 10V, X7R -> 6.3V, X5R
- C202: footprint Capacitor_SMD:C_1206_3216Metric -> Capacitor_SMD:C_0805_2012Metric; Rating 10V, X7R -> 6.3V, X5R
- D201: value DF3A5.6LFU -> PESD3V3S2UT; footprint Package_TO_SOT_SMD:SOT-323_SC-70 -> Package_TO_SOT_SMD:SOT-23; LCSC (none) -> C84276
- J201: Alternative (none) -> GT-USB-7010ASV; LCSC (none) -> C2988369
- J202: LCSC (none) -> C41431904
- RN201: LCSC (none) -> C2654032
- SW201: value EVQ-P7A01P -> EVQ-P7J01P; symbol EVQ-P7A01P:EVQ-P7A01P -> EVQ-P7A01P:EVQ-P7J01P; Alternative (none) -> EVQ-PJA01P; Availability In Stock -> (none); Check_prices https://www.snapeda.com/parts/EVQ-P7A01P/Panasonic+Electron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 -> (none); Description_1 Tactile Switch SPST-NO Side Actuated Surface Mount, Right A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 -> (none); LCSC (none) -> C2828254; MANUFACTURER Panasonic Electronic Components -> (none); MP EVQ-P7A01P -> EVQ-P7J01P; PARTREV 2022.4 -> (none); Package None -> (none); Price None -> (none); STANDARD Manufacturer Recommendations -> (none); SnapEDA_Link https://www.snapeda.com/parts/EVQ-P7A01P/Panasonic+Electron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 -> (none)
- SW202: value EVQ-P7A01P -> EVQ-P7J01P; symbol EVQ-P7A01P:EVQ-P7A01P -> EVQ-P7A01P:EVQ-P7J01P; Alternative (none) -> EVQ-P7A01P; Availability In Stock -> (none); Check_prices https://www.snapeda.com/parts/EVQ-P7A01P/Panasonic+Electron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 -> (none); Description_1 Tactile Switch SPST-NO Side Actuated Surface Mount, Right A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 -> (none); LCSC (none) -> C2828254; MANUFACTURER Panasonic Electronic Components -> (none); MP EVQ-P7A01P -> EVQ-P7J01P; PARTREV 2022.4 -> (none); Package None -> (none); Price None -> (none); STANDARD Manufacturer Recommendations -> (none); SnapEDA_Link https://www.snapeda.com/parts/EVQ-P7A01P/Panasonic+Electron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 -> (none)
- U201: value TCA9555RTWR -> TCA9555RTW; LCSC (none) -> C140277
- U202: value ESP32-C3-WROOM-02 -> ESP32-C3-WROOM-02-N4; LCSC (none) -> C2934560
Connections:
- net SCL: now also U201.19 (SCL); no longer U201.20 (SDA)
- net SDA: now also U201.20 (SDA); no longer U201.19 (SCL)
Other:
- note added: "A great place to plug in off-the-shelf accessories - Host has pull-ups so accessories don't need their own - 3.3 V supply is regulated, 600 mA current available"
- note removed: "Host has pull-ups so accessories don't need their own"
