File: hardware/minuet/v2/fan.kicad_sch (KiCad schematic)
At the start: 25 parts, among them J301 B3P-VH-B, J302 B5B-XH-A, U301 MCT8315Z0HRRYR

Commit message: Finalize Minuet v2.1 for manufacture.
This revision uses a different motor controller and buck converter
and remedies errata from v2.0.
Parts:
- C301: value 10u -> 22u; footprint Capacitor_SMD:C_1206_3216Metric -> Capacitor_SMD:C_0805_2012Metric; Rating 25V, X7R -> 25V, X5R
- C302, C305: Rating 25V, X7R -> 25V, X5R
- C303: Rating 16V, X7R -> 16V, X5R
- C304: footprint Capacitor_SMD:C_1206_3216Metric -> Capacitor_SMD:C_0805_2012Metric; Rating 10V, X7R -> 6.3V, X5R
- C306, C307: Rating 10V, X7R -> 6.3V, X5R
- J301: LCSC (none) -> C265360
- J302: LCSC (none) -> C157991
- R301, R303: value 10K -> 18.2K
- R302: value 3.40K -> 3.65K
- R309: now not fitted; now left out of the parts list
- R310, R311: now fitted
- R312: now left out of the parts list
- RV301: LCSC (none) -> C81260
- U301: value MCT8315Z0HRRYR -> MCT8316Z0T; footprint MCT8315Z:IC_MCT8315Z0HRRYR -> MCT8316Z:MCT8316ZT; symbol MCT8315Z0HRRYR:MCT8315Z0HRRYR -> MCT8316ZT:MCT8316ZT; Description_1 40-V max, 4-A peak, sensored trapezoidal control 3-phase BL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 -> 40-V max, 8-A peak, sensored trapezoidal control 3-phase BL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; LCSC (none) -> C3681342; MP MCT8315Z0HRRYR -> MCT8316Z0TRGFR
Connections:
- net +12V: now also U301.10 (VM), U301.11 (VM); no longer U301.8 (VM)
- net ADVANCE: now also U301.35 (ADVANCE); no longer U301.28 (ADVANCE)
- net AVDD: now also U301.25 (AVDD); no longer U301.19 (AVDD)
- net DIR: now also U301.36 (DIR); no longer U301.29 (DIR)
- net GND: now also U301.12 (PGND), U301.2 (AGND), U301.21 (DRVOFF), U301.26 (AGND), U301.4 (GND_BK); no longer U301.10 (PGND), U301.14 (PGND), U301.3 (GND_BK), U301.31 (BRAKE), U301.33 (EP), U301.34 (EP), U301.35 (EP), U301.36 (EP), U301.37 (EP), U301.39 (EP), U301.40 (EP), U301.42 (EP), U301.43 (EP), U301.44 (EP)
- net ILIM: now also U301.37 (ILIM); no longer U301.30 (ILIM)
- net MODE: now also U301.33 (MODE); no longer U301.26 (MODE)
- net NFAULT: now also U301.22 (~{FAULT}); no longer U301.16 (~{FAULT})
- net NSLEEP: now also U301.23 (~{SLEEP}); no longer U301.17 (~{SLEEP})
- net PWM: now also U301.39 (PWM); no longer U301.32 (PWM)
- net SLEW: now also U301.34 (SLEW); no longer U301.27 (SLEW)
- net TACH: now also U301.40 (FGOUT); no longer U301.1 (FGOUT)
- net U: now also U301.13 (OUTA), U301.14 (OUTA); no longer U301.11 (OUTA)
- net U_HALL: now also U301.27 (HPA); no longer U301.20 (HPA)
- net V: now also U301.16 (OUTB), U301.17 (OUTB); no longer U301.12 (OUTB)
- net VBK: now also U301.3 (FB_BK); no longer U301.2 (FB_BK)
- net V_HALL: now also U301.29 (HPB); no longer U301.22 (HPB)
- net W: now also U301.19 (OUTC), U301.20 (OUTC); no longer U301.13 (OUTC)
- net W_HALL: now also U301.31 (HPC); no longer U301.24 (HPC)
- net at L301.2: now also U301.5 (SW_BK); no longer U301.4 (SW_BK)
- net at C303.2: now also U301.8 (CP); no longer U301.7 (CP)
- net at C305.2: now also U301.6 (CPL); no longer U301.5 (CPL)
- net at C305.1: now also U301.7 (CPH); no longer U301.6 (CPH)
- no-connect marks 3 -> 4
Other:
- note added: "Commutation advance lead angle - 0°: tied to AGND (default) - 4°: tied to AGND via 22 Kohm resistor - 11°: tied to AGND via 100 Kohm resistor - 15°: Hi-Z - 20°: tied to AVDD via 100 Kohm resistor - 25°: tied to AVDD via 22 Kohm resistor - 30°: tied to AVDD"
- note added: "Current limit setting for sum of all phases - Assume CSA_GAIN = 0.15 V/A, V(AVDD) = 3.3 V - Calculate Ilim Ilim = V(AVDD) * (0.5 - RF / (2 * RF + RV)) / CSA_GAIN * 3 Ilim = 66 A * (0.5 - RF / (2 * RF + RV)) - Choose RF so that Ilim_max = 4 A with RV_max = 5 K RF = 18.2 Kohm - Calculate RV for given Ilim RV = RF * (1 / (0.5 - Ilim / 66 A) - 2) Approximate setpoints rounded to nearest E96 series va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"
- note added: "Increasing resistance of the setpoint increases the current limit Specified to a maximum of 4 A"
- note added: "Slew rate control - 25 V/uS: tied to AGND - 50 V/uS: Hi-Z - 100 V/uS: tied to AVDD via 47 Kohm resistor - 200 V/uS: connected to AVDD (default)"
- note removed: "Commutation advance phase angle - 0°: tied to AGND - 4°: tied to AGND via 22 Kohm resistor - 11°: tied to AGND via 100 Kohm resistor - 15°: Hi-Z - 20°: tied to AVDD via 100 Kohm resistor - 25°: tied to AVDD via 22 Kohm resistor - 30°: tied to AVDD (default)"
- note removed: "Current limit setting - Vilim = AVDD/2 - 0.08 V/A * Ilim, where AVDD/2 = 1.65 V - Disabled when Ilim = 0 A - Accuracy is 14% when Ilim > 1A - Ilim = 20.625 A - 41.25 A/Kohm * (10 Kohm / (20 Kohm + RV(Kohm))) Approximate setpoints - Ilim = 0 A (disabled) => RV = 0 K - Ilim = 1.5 A => RV = 1.58 K - Ilim = 2 A => RV = 2.15 K - Ilim = 2.5 A => RV = 2.80 K - Ilim = 3 A => RV = 3.40 K - Ilim = 3.5 A =>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"
- note removed: "Increasing resistance of the setpoint increases the current limit"
- note removed: "Slew rate control - 25 V/uS: tied to AGND - 50 V/uS: Hi-Z (default) - 100 V/uS: tied to AVDD via 47 Kohm resistor - 200 V/uS: connected to AVDD"
- moved on the sheet: C306, R301, R302, R303, RV301, TP301

Commit message: Update Minuet v2.2 ILIM resistor setting.
The default current limits are just a little too low, fix that in
the next revision.  Also improved the documentation with markdown tables
for each setting.
Parts:
- R301, R303: value 18.2K -> 14K
Other:
- note added: "Current limit setting for sum of all phases - Assume CSA_GAIN = 0.15 V/A, V(AVDD) = 3.3 V - Calculate Ilim Ilim = V(AVDD) * (0.5 - RF / (2 * RF + RV)) / CSA_GAIN * 3 Ilim = 66 A * (0.5 - RF / (2 * RF + RV)) - Choose RF so that Ilim_max = 5 A with RV_max = 5 K (allows tolerance for the default 4 A setting and a little extra beyond it) RF = 14 Kohm - Calculate RV for given Ilim RV = RF * (1 / (0.5 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"
- note added: "Increasing resistance of the setpoint increases the current limit Specified to a maximum of 5 A (default of 4 A)"
- note removed: "Current limit setting for sum of all phases - Assume CSA_GAIN = 0.15 V/A, V(AVDD) = 3.3 V - Calculate Ilim Ilim = V(AVDD) * (0.5 - RF / (2 * RF + RV)) / CSA_GAIN * 3 Ilim = 66 A * (0.5 - RF / (2 * RF + RV)) - Choose RF so that Ilim_max = 4 A with RV_max = 5 K RF = 18.2 Kohm - Calculate RV for given Ilim RV = RF * (1 / (0.5 - Ilim / 66 A) - 2) Approximate setpoints rounded to nearest E96 series va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"
- note removed: "Increasing resistance of the setpoint increases the current limit Specified to a maximum of 4 A"
Changed lines of the file:
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@@
 	(rectangle
 		(start 182.88 13.97)
-		(end 267.97 110.49)
+		(end 267.97 123.19)
 		(stroke
 			(width 0)
@@
 		)
 	)
-	(text "Increasing resistance of the setpoint increases the current limit\nSpecified to a maximum of 4 A"
+	(text "Increasing resistance of the setpoint increases the current limit\nSpecified to a maximum of 5 A (default of 4 A)"
 		(exclude_from_sim no)
 		(at 184.15 19.05 0)
@@
 		)
 	)
-	(text "Current limit setting for sum of all phases\n- Assume CSA_GAIN = 0.15 V/A, V(AVDD) = 3.3 V\n- Calculate Ilim\n    Ilim = V(AVDD) * (0.5 - RF / (2 * RF + RV)) / CSA_GAIN * 3\n    Ilim = 66 A * (0.5 - RF / (2 * RF + RV))\n- Choose RF so that Ilim_max = 4 A with RV_max = 5 K\n    RF = 18.2 Kohm\n- Calculate RV for given Ilim\n    RV = RF * (1 / (0.5 - Ilim / 66 A) - 2)\n\nApproximate setpoints rounded to nearest E96 series value\n- Ilim = 0 A (disabled) => RV = 0 K\n- Ilim = 1 A => RV = 1.13 K\n- Ilim = 1.5 A => RV = 1.74 K\n- Ilim = 2 A => RV = 2.32 K\n- Ilim = 2.5 A => RV = 3.00 K\n- Ilim = 3 A => RV = 3.65 K (default)\n- Ilim = 3.5 A => RV = 4.32 K\n- Ilim = 4 A (maximum) => RV = 4.99 K\n"
+	(text "Current limit setting for sum of all phases\n- Assume CSA_GAIN = 0.15 V/A, V(AVDD) = 3.3 V\n- Calculate Ilim\n    Ilim = V(AVDD) * (0.5 - RF / (2 * RF + RV)) / CSA_GAIN * 3\n    Ilim = 66 A * (0.5 - RF / (2 * RF + RV))\n- Choose RF so that Ilim_max = 5 A with RV_max = 5 K\n   (allows tolerance for the default 4 A setting and a little extra beyond it)\n    RF = 14 Kohm\n- Calculate RV for given Ilim\n    RV = RF * (1 / (0.5 - Ilim / 66 A) - 2)\n\nApproximate setpoints rounded to nearest E96 series value\n- Ilim = 0 A => RV = 0 K (disabled)\n- Ilim = 1 A => RV = 0.887 K\n- Ilim = 1.5 A => RV = 1.33 K\n- Ilim = 2 A => RV = 1.82 K\n- Ilim = 2.5 A => RV = 2.32 K\n- Ilim = 3 A => RV = 2.80 K\n- Ilim = 3.5 A => RV = 3.32 K\n- Ilim = 4 A => RV = 3.83 K (default)\n- Ilim = 4.5 A => RV = 4.42 K\n- Ilim = 5 A => RV = 4.99 K (maximum)\n\nMeasurement at the bench shows average motor phase current about 75%\nof the value configured by ILIM at full duty cycle."
 		(exclude_from_sim no)
 		(at 187.96 69.85 0)
@@
 			)
 		)
-		(property "Value" "18.2K"
+		(property "Value" "14K"
 			(at 203.2 29.1296 90)
 			(effects
@@
 			)
 		)
-		(property "Value" "18.2K"
+		(property "Value" "14K"
 			(at 240.538 53.34 0)
 			(effects
