File: hardware/light/v3/light.kicad_sch (KiCad schematic)
At the start: 18 parts, among them J1 PH2-16-UA, J2 Conn_01x09, J3 Conn_01x09, J4 B3B-XH-A, Q1 DMG2301L, Q2 MMBT3904, U1 LP2985-50DBVR, U2 SN74LVC1G17DBVR

Commit message: Add a connector for input controls.
Parts:
- added C4, C5: 10n, Capacitor_SMD:C_0603_1608Metric, symbol Device:C
- added J5: B5B-XH-A, Connector_JST:JST_XH_B5B-XH-A_1x05_P2.50mm_Vertical, symbol Connector_Generic:Conn_01x05
- added R7: 10K, Resistor_SMD:R_0603_1608Metric, symbol Device:R
- added R8, R9: 100K, Resistor_SMD:R_0603_1608Metric, symbol Device:R
- added RV1: 10K, symbol Device:R_Potentiometer
- added SW1: SW_Push, symbol Switch:SW_Push
- C1, C2: Rating 25V, X5R -> 50V, X5R
- C3: Rating 6.3V, X5R -> 16V, X5R
- J2, J3: now left out of the parts list
- Q1: Rating (none) -> -20V, -3A
Connections:
- net +3.3V: now also C4.2, C5.2, J5.5 (Pin_5), R7.1, R8.2, R9.2
- net GND: now also J5.1 (Pin_1), RV1.3, SW1.2
- net GPIO0: now also C4.1, J5.2 (Pin_2), R8.1, RV1.2
- net GPIO1: now also C5.1, J5.4 (Pin_4), R9.1, SW1.1
- net GPIO5: now also R6.2, U2.2; no longer R3.2
- net GPIO6: now also R3.2; no longer R6.2, U2.2
- new net PH: J5.3 (Pin_3), R7.2, RV1.1
Other:
- note added: "5 V LEVEL SHIFTER FOR DATA"
- note added: "Controls the light intensity, mode, or other functions, connect the input devices as indicated Potentiometer input: Connect a 10 Kohm pressure-sensitive strip (e.g. "ThinPot" or "SoftPot") or an ordinary potentiometer Switch input: Leave unconnected when using a pressure-sensitive strip, otherwise connect a momentary push-button Alternatively, the inputs could be used for a rotary encoder"
- note added: "HIGH-SIDE SWITCH FOR 1 A LOAD AT 12 V"
- note added: "OUTPUT CONNECTOR FOR LOAD AND DATA"
- note added: "POTENTIOMETER AND SWITCH INPUT"
- note added: "Suitable for PWM dimmable LED light or addressable LED strip"
- note removed: "5 V level shifter"
- note removed: "High side P-Channel MOSFET for resistive load up to 1 A"
- note removed: "Output connector for load and data"
- note removed: "Suitable for dimmable LED light or addressable LED strip"
- company: (none) -> Brown Studios LLC
- moved on the sheet: C1, C2, C3, J1, J2, J3, J4, JP1, Q1, Q2, R1, R2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

Commit message: Finalize light accessory for fabrication.
Parts:
- removed C4, C5: 10n, Capacitor_SMD:C_0603_1608Metric, symbol Device:C
- removed J5: B5B-XH-A, Connector_JST:JST_XH_B5B-XH-A_1x05_P2.50mm_Vertical, symbol Connector_Generic:Conn_01x05
- removed R7: 10K, Resistor_SMD:R_0603_1608Metric, symbol Device:R
- removed R8, R9: 100K, Resistor_SMD:R_0603_1608Metric, symbol Device:R
- removed RV1: 10K, symbol Device:R_Potentiometer
- removed SW1: SW_Push, symbol Switch:SW_Push
Other:
- note removed: "Controls the light intensity, mode, or other functions, connect the input devices as indicated Potentiometer input: Connect a 10 Kohm pressure-sensitive strip (e.g. "ThinPot" or "SoftPot") or an ordinary potentiometer Switch input: Leave unconnected when using a pressure-sensitive strip, otherwise connect a momentary push-button Alternatively, the inputs could be used for a rotary encoder"
- note removed: "POTENTIOMETER AND SWITCH INPUT"
- moved on the sheet: C1, C2, C3, J1, J2, J3, J4, JP1, Q1, Q2, R1, R2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

Commit message: Add tooling holes and PCBA offsets.
Parts:
- J1: FT Rotation Offset (none) -> -90
Changed lines of the file:
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@@
+			)
+		)
+		(property "FT Rotation Offset" "-90"
+			(at 74.93 93.98 0)
+			(effects
+				(font
+					(size 1.27 1.27)
+				)
+				(hide yes)
 			)
 		)

Commit message: Prepare light accessory v3 for production
Parts:
- J1: Alternative (none) -> 10129381-916001BLF
- U1: LCSC LP2985-50DBVR -> C74511
- U2: LCSC SN74LVC1G17DBVR -> C7836
Changed lines of the file:
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@@
 			)
 		)
-		(property "LCSC" "LP2985-50DBVR"
+		(property "LCSC" "C74511"
 			(at 146.05 68.58 0)
 			(effects
@@
 			)
 		)
+		(property "Alternative" "10129381-916001BLF"
+			(at 74.93 93.98 0)
+			(effects
+				(font
+					(size 1.27 1.27)
+				)
+				(hide yes)
+			)
+		)
 		(pin "4"
 		)
@@
 			)
 		)
-		(property "LCSC" "SN74LVC1G17DBVR"
+		(property "LCSC" "C7836"
 			(at 151.13 118.11 0)
 			(effects
