File: hardware/minuet/v3/core.kicad_sch (KiCad schematic)
At the start: 15 parts, among them J201 USB4105-GF-A, J202 SM04B-SRSS-TB, SW201 EVQ-P7J01P, SW202 EVQ-P7J01P, U201 TCA9555RTW, U202 ESP32-C3-WROOM-02-N4

Commit message: First draft of Minuet v3.
Parts:
- removed RN201: 746X101103JP, 746X:RESCAXS64P320X160X70-10N, symbol 746X:746X101nnnJP
- added R17, R19, R21, R22, R23: 10K, Resistor_SMD:R_0603_1608Metric, symbol Device:R
- renumbered C203 to C10, C204 to C11, C205 to C12, C201 to C8, C202 to C9, D201 to D2, J201 to J6, J202 to J7, R201 to R18, R202 to R20, SW201 to SW1, SW202 to SW2, U201 to U3, U202 to U4
Connections:
- net GPIO8_STRAP is gone; now on net SCL: U4.7 (GPIO8)
- net +3.3V: now also R17.2, R19.2, R21.2, R22.2, R23.2
- net BOOT: now also R17.1
- net GPIO2_STRAP: now also R21.1
- net RESET: now also R19.1
- net SCL: now also R22.1; no longer U4.5 (GPIO6)
- net SDA: now also R23.1
- new net GPIO6: U4.5 (GPIO6)
- no-connect marks 6 -> 4
Other:
- moved on the sheet: J7

Commit message: Prepare for fabrication.
Parts:
- C10, C8: LCSC (none) -> C14663
- C11: LCSC (none) -> C1634
- C12: LCSC (none) -> C15849
- C9: LCSC (none) -> C15850
- J6: FT Position Offset (none) -> 0,1.27
- J7: Alternative (none) -> GT-A1002WRS-104SBT01; LCSC C41431904 -> C160404; LCSC_Alternative (none) -> C41431904
- R17, R19, R21, R22, R23: LCSC (none) -> C25804
- R18, R20: LCSC (none) -> C23186
- SW1: value EVQ-P7J01P -> EVQ-P7A01P; Alternative EVQ-PJA01P -> EVQ-P7J01P; LCSC C2828254 -> C79167; LCSC_Alternative (none) -> C2828254; MP EVQ-P7J01P -> (none)
- SW2: value EVQ-P7J01P -> EVQ-P7A01P; Alternative EVQ-P7A01P -> EVQ-P7J01P; LCSC C2828254 -> C79167; LCSC_Alternative (none) -> C2828254; MP EVQ-P7J01P -> (none)
- U3: FT Rotation Offset (none) -> 270

Commit message: Remove unnecessary fields.
Parts:
- SW1, SW2: MAXIMUM_PACKAGE_HEIGHT 1.35mm -> (none); MF Panasonic Electronic -> (none)

Commit message: Prepare Minuet v3 for production.
Parts:
- C10, C8, C9: Rating 6.3V, X5R -> 50V, X5R
- C11: LCSC C1634 -> C1634; Rating 6.3V, X5R -> 50V, X5R
- C12: LCSC C15849 -> C15849; Rating 6.3V, X5R -> 50V, X5R
- SW1, SW2: footprint EVQ-P7A01P:SW_EVQ-P7A01P -> Button_Switch_SMD:SW_SPST_EVQP7A; symbol EVQ-P7A01P:EVQ-P7J01P -> Switch:SW_SPST
Connections:
- net BOOT: now also SW1.1 (A); no longer SW1.1_1, SW1.1_2
- net GND: now also SW1.2 (B), SW2.2 (B); no longer SW1.2_1, SW1.2_2, SW2.2_1, SW2.2_2
- net RESET: now also SW2.1 (A); no longer SW2.1_1, SW2.1_2
Other:
- moved on the sheet: C11, C12
