File: hardware/minuet/v3/fan.kicad_sch (KiCad schematic)
At the start: 25 parts, among them J301 B3P-VH-B, J302 B5B-XH-A, U301 MCT8316Z0T

Commit message: First draft of Minuet v3.
Parts:
- removed C304: 22u, Capacitor_SMD:C_0805_2012Metric, symbol Device:C
- removed C306: 100n, Capacitor_SMD:C_0603_1608Metric, symbol Device:C
- removed J302: B5B-XH-A, Connector_JST:JST_XH_B5B-XH-A_1x05_P2.50mm_Vertical, symbol Connector_Generic:Conn_01x05
- removed L301: 22u, Inductor_SMD:L_0603_1608Metric, symbol Device:L_Small
- removed R301, R303: 14K, Resistor_SMD:R_0603_1608Metric, symbol Device:R
- removed R302: 3.65K, Resistor_SMD:R_0603_1608Metric_Pad0.98x0.95mm_HandSolder, symbol Device:R
- removed R304, R305, R306: 4.7K, Resistor_SMD:R_0603_1608Metric, symbol Device:R
- removed R307, R309, R310, R311, R312: 0R, Resistor_SMD:R_0603_1608Metric_Pad0.98x0.95mm_HandSolder, symbol Device:R
- removed R308: 22K, Resistor_SMD:R_0603_1608Metric_Pad0.98x0.95mm_HandSolder, symbol Device:R
- removed RV301: 5K, 3362P-1-502LF:TRIM_3362P-1-502LF, symbol Device:R_Potentiometer_Trim
- removed TP301: TestPoint_2Pole, TestPoint:TestPoint_2Pads_Pitch2.54mm_Drill0.8mm, symbol Connector:TestPoint_2Pole
- added C18: 1u, Capacitor_SMD:C_0603_1608Metric, symbol Device:C
- C17: renamed from C307; Rating 6.3V, X5R -> 10V, X5R
- U5: renamed from U301; value MCT8316Z0T -> MCF8316D; footprint MCT8316Z:MCT8316ZT -> MCF8316D:MCF8316D; symbol MCT8316ZT:MCT8316ZT -> MCF8316D:MCF8316D; Availability In Stock -> (none); Check_prices https://www.snapeda.com/parts/MCT8315Z0HRRYR/Texas+Instrume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 -> (none); Description_1 40-V max, 8-A peak, sensored trapezoidal control 3-phase BL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 -> Sensorless Field Oriented Control (FOC) Integrated FET BLDC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; LCSC C3681342 -> (none); MP MCT8316Z0TRGFR -> MCF8316DVRGFR; PARTREV December 2023 -> May 2025; STANDARD Manufacturer Recommendations -> (none); SnapEDA_Link https://www.snapeda.com/parts/MCT8315Z0HRRYR/Texas+Instrume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 -> (none)
- renumbered C301 to C13, C302 to C14, C303 to C15, C305 to C16, J301 to J8
Connections:
- net ADVANCE is gone; now on net GND: U5.35 (BRAKE)
- net MODE is gone; now on net GND: U5.33 (EXT_CLK)
- net NSLEEP is gone; now on net GND: U5.23 (NC)
- net SLEW is gone; now on net GND: U5.34 (DIR)
- net TACH is gone; now on net NFAULT: U5.40 (~{FAULT})
- net U_HALL is gone; now on an unnamed net: U5.27 (AVDD)
- net GND: now also U5.22 (NC), U5.24 (NC), U5.25 (NC), U5.32 (EXT_WD), C18.2; no longer U5.38 (BRAKE)
- net NFAULT: no longer U5.22 (~{FAULT})
- net at U5.1 (DVDD): now also C18.1
- net WAKE: now reaches U5.28 (SPEED/WAKE)
- net SDA: now reaches U5.30 (SDA)
- net AVDD: no longer names the net of C17.1
- net AVDD: no longer U5.25 (AVDD)
- net DIR: no longer names the net of U5.36 (DACOUT1)
- net ILIM: no longer names the net of U5.37 (DACOUT2)
- net PWM: no longer names the net of U5.39 (ALARM)
- net U renamed A
- net V renamed B
- net VBK renamed +3.3V
- net V_HALL: no longer names the net of U5.29 (FG)
- net W renamed C
- net W_HALL renamed SCL
- no-connect marks 4 -> 6
Other:
- note added: "AVDD supplies 3.3 V for internal analog circuitry from VM when not sleeping DVDD supplies 1.5 V for internal digital logic from FB_BK when not sleeping FB_BK is externally powered with 3.3 V and the buck converter is disabled to reduce BOM cost per application note SLLA643 NFAULT is open-drain, has an internal pull-up to AVDD that can be disabled via I2C, SLLA643 says never use external and inter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"
- note removed: "AVDD supplies 20 mA @ 3.3 V derived from VM when NSLEEP is active SW_BK supplies 50 mA @ 5 V from a built-in buck converter NFAULT is open-drain, must be high on reset to not enter test mode TACH/FGOUT is open-drain, pulses with each hall sensor transition Internal pull-down on NSLEEP, BRAKE, DIR, PWM, DRVOFF"
- note removed: "COMMUTATION ADVANCE"
- note removed: "COMMUTATION MODE"
- note removed: "CURRENT LIMIT"
- note removed: "Commutation advance lead angle - 0°: tied to AGND (default) - 4°: tied to AGND via 22 Kohm resistor - 11°: tied to AGND via 100 Kohm resistor - 15°: Hi-Z - 20°: tied to AVDD via 100 Kohm resistor - 25°: tied to AVDD via 22 Kohm resistor - 30°: tied to AVDD"
- note removed: "Current limit setting for sum of all phases - Assume CSA_GAIN = 0.15 V/A, V(AVDD) = 3.3 V - Calculate Ilim Ilim = V(AVDD) * (0.5 - RF / (2 * RF + RV)) / CSA_GAIN * 3 Ilim = 66 A * (0.5 - RF / (2 * RF + RV)) - Choose RF so that Ilim_max = 5 A with RV_max = 5 K (allows tolerance for the default 4 A setting and a little extra beyond it) RF = 14 Kohm - Calculate RV for given Ilim RV = RF * (1 / (0.5 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"
- note removed: "Increasing resistance of the setpoint increases the current limit Specified to a maximum of 5 A (default of 4 A)"
- note removed: "Mode - Type 2: tied to AGND via 22 Kohm resistor - digital hall input - asynchronous modulation - ASR & AAR disabled - Type 4: Hi-Z - digital hall input - synchronous modulation - ASR & AAR disabled - Type 7: tied to AVDD (default) - digital hall input - synchronous modulation - ASR & AAR enabled"
- note removed: "SLEW RATE"
- note removed: "Slew rate control - 25 V/uS: tied to AGND - 50 V/uS: Hi-Z - 100 V/uS: tied to AVDD via 47 Kohm resistor - 200 V/uS: connected to AVDD (default)"
- moved on the sheet: C13, C14, C15, C16, C17, J8

Commit message: Prepare for fabrication.
Parts:
- C13: LCSC (none) -> C45783
- C14: LCSC (none) -> C14663
- C15, C17, C18: LCSC (none) -> C15849
- C16: LCSC (none) -> C1622
- U5: FT Rotation Offset (none) -> 270; LCSC (none) -> C42453588

Commit message: Remove unnecessary fields.
Parts:
- U5: Description_1 Sensorless Field Oriented Control (FOC) Integrated FET BLDC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 -> (none); MANUFACTURER Texas Instruments -> (none); MAXIMUM_PACKAGE_HEIGHT 0.8mm -> (none); MF Texas Instruments -> (none); MP MCF8316DVRGFR -> (none); PARTREV May 2025 -> (none); Package None -> (none); Price None -> (none)

Commit message: Prepare Minuet v3 for production.
Parts:
- C14, C16: Rating 25V, X5R -> 50V, X5R
- C15: LCSC C15849 -> C15849; Rating 16V, X5R -> 50V, X5R
- C17, C18: LCSC C15849 -> C15849; Rating 10V, X5R -> 50V, X5R
- U5: LCSC C42453588 -> C42453588
Other:
- moved on the sheet: C13, C14, C15, C16, C17, C18, J8, U5
