File: hardware/minuet/v3/keypad.kicad_sch (KiCad schematic)
At the start: 3 parts, among them J501 G800LE300018YEU, J502 MTJ-889X1, J503 MTJ-669X1

Commit message: First draft of Minuet v3.
Parts:
- renumbered J501 to J10, J502 to J11, J503 to J12
Other:
- note added: "Compatible with original equipment Key matrix - R1+GND: Close lid - R2+GND: Open lid - R1+C1: Fan off - R1+C2: Fan speed up - R1+C3: Fan speed down - R1+C2+C3: Open / close lid - R1+C4: Toggle rain sensor (only certain models) - R2+C1: Fan on and cycle speeds - R2+C2: Fan on / off - R2+C3: Fan intake / exhaust direction - R2+C4: Toggle auto thermostat LEDs - LED_AUTO: Auto LED cathode, green with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"
- note removed: "Compatible with original equipment Key matrix - R1+GND: Close cover - R2+GND: Open cover - R1+C1: Fan off - R1+C2: Fan speed up - R1+C3: Fan speed down - R1+C2+C3: Open / close cover - R1+C4: Toggle rain sensor (only certain models) - R2+C1: Fan on and cycle speeds - R2+C2: Fan on / off - R2+C3: Fan intake / exhaust direction - R2+C4: Toggle auto thermostat LEDs - LED_AUTO: Auto LED cathode, gree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"
Changed lines of the file:
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@@
 		)
 	)
-	(text "Compatible with original equipment\n\nKey matrix\n- R1+GND: Close cover\n- R2+GND: Open cover\n- R1+C1: Fan off\n- R1+C2: Fan speed up\n- R1+C3: Fan speed down\n- R1+C2+C3: Open / close cover\n- R1+C4: Toggle rain sensor (only certain models)\n- R2+C1: Fan on and cycle speeds\n- R2+C2: Fan on / off\n- R2+C3: Fan intake / exhaust direction\n- R2+C4: Toggle auto thermostat\n\nLEDs\n- LED_AUTO: Auto LED cathode, green with 2.4 V voltage drop\n- LED_RAIN: Rain LED cathode, red (only certain models)\n\nKEY_Rx and KEY_Cx inputs need pull-ups\nDetect key press when KEY_Rx goes low when undriven (tristate)\nDetect key press when KEY_Cx goes low during high-to-low strobe of KEY_Rx\nFan originally provided +5V supply the interface but +3.3V works fine"
+	(text "Compatible with original equipment\n\nKey matrix\n- R1+GND: Close lid\n- R2+GND: Open lid\n- R1+C1: Fan off\n- R1+C2: Fan speed up\n- R1+C3: Fan speed down\n- R1+C2+C3: Open / close lid\n- R1+C4: Toggle rain sensor (only certain models)\n- R2+C1: Fan on and cycle speeds\n- R2+C2: Fan on / off\n- R2+C3: Fan intake / exhaust direction\n- R2+C4: Toggle auto thermostat\n\nLEDs\n- LED_AUTO: Auto LED cathode, green with 2.4 V voltage drop\n- LED_RAIN: Rain LED cathode, red (only certain models)\n\nKEY_Rx and KEY_Cx inputs need pull-ups\nDetect key press when KEY_Rx goes low when undriven (tristate)\nDetect key press when KEY_Cx goes low during high-to-low strobe of KEY_Rx\nFan originally provided +5V supply the interface but +3.3V works fine"
 		(exclude_from_sim no)
 		(at 95.25 59.69 0)
@@
 		(dnp no)
 		(fields_autoplaced yes)
-		(property "Reference" "#PWR0502"
+		(property "Reference" "#PWR069"
 			(at 116.84 121.92 0)
 			(effects
@@
 			(project "minuet"
 				(path "/5bd7983a-3caa-4bb2-9dc5-1af533f31e50/ecd3cea2-5b83-45e6-bc3a-38348e0ff880"
-					(reference "#PWR0502")
+					(reference "#PWR069")
 					(unit 1)
 				)
@@
 		(on_board yes)
 		(dnp no)
-		(property "Reference" "J503"
+		(property "Reference" "J12"
 			(at 204.724 111.252 0)
 			(effects
@@
 			(project "minuet"
 				(path "/5bd7983a-3caa-4bb2-9dc5-1af533f31e50/ecd3cea2-5b83-45e6-bc3a-38348e0ff880"
-					(reference "J503")
+					(reference "J12")
 					(unit 1)
 				)
@@
 		(on_board yes)
 		(dnp no)
-		(property "Reference" "J502"
+		(property "Reference" "J11"
 			(at 160.02 110.236 0)
 			(effects
@@
 			(project "minuet"
 				(path "/5bd7983a-3caa-4bb2-9dc5-1af533f31e50/ecd3cea2-5b83-45e6-bc3a-38348e0ff880"
-					(reference "J502")
+					(reference "J11")
 					(unit 1)
 				)
@@
 		(dnp no)
 		(fields_autoplaced yes)
-		(property "Reference" "#PWR0503"
+		(property "Reference" "#PWR070"
 			(at 151.13 121.92 0)
 			(effects
@@
 			(project "minuet"
 				(path "/5bd7983a-3caa-4bb2-9dc5-1af533f31e50/ecd3cea2-5b83-45e6-bc3a-38348e0ff880"
-					(reference "#PWR0503")
+					(reference "#PWR070")
 					(unit 1)
 				)
@@
 		(dnp no)
 		(fields_autoplaced yes)
-		(property "Reference" "#PWR0504"
+		(property "Reference" "#PWR071"
 			(at 185.42 127 0)
 			(effects
@@
 			(project "minuet"
 				(path "/5bd7983a-3caa-4bb2-9dc5-1af533f31e50/ecd3cea2-5b83-45e6-bc3a-38348e0ff880"
-					(reference "#PWR0504")
+					(reference "#PWR071")
 					(unit 1)
 				)
@@
 		(dnp no)
 		(fields_autoplaced yes)
-		(property "Reference" "#PWR0501"
+		(property "Reference" "#PWR068"
 			(at 195.58 119.38 0)
 			(effects
@@
 			(project "minuet"
 				(path "/5bd7983a-3caa-4bb2-9dc5-1af533f31e50/ecd3cea2-5b83-45e6-bc3a-38348e0ff880"
-					(reference "#PWR0501")
+					(reference "#PWR068")
 					(unit 1)
 				)
@@
 		(on_board yes)
 		(dnp no)
-		(property "Reference" "J501"
+		(property "Reference" "J10"
 			(at 110.998 110.236 0)
 			(effects
@@
 			(project "minuet"
 				(path "/5bd7983a-3caa-4bb2-9dc5-1af533f31e50/ecd3cea2-5b83-45e6-bc3a-38348e0ff880"
-					(reference "J501")
+					(reference "J10")
 					(unit 1)
 				)

Commit message: Prepare Minuet v3 for production.
Parts:
- J10: Alternative (none) -> 0022284081; LCSC_Alternative (none) -> C3339252
Changed lines of the file:
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@@
 		)
 	)
-	(text "Compatible with original equipment\n\nKey matrix\n- R1+GND: Close lid\n- R2+GND: Open lid\n- R1+C1: Fan off\n- R1+C2: Fan speed up\n- R1+C3: Fan speed down\n- R1+C2+C3: Open / close lid\n- R1+C4: Toggle rain sensor (only certain models)\n- R2+C1: Fan on and cycle speeds\n- R2+C2: Fan on / off\n- R2+C3: Fan intake / exhaust direction\n- R2+C4: Toggle auto thermostat\n\nLEDs\n- LED_AUTO: Auto LED cathode, green with 2.4 V voltage drop\n- LED_RAIN: Rain LED cathode, red (only certain models)\n\nKEY_Rx and KEY_Cx inputs need pull-ups\nDetect key press when KEY_Rx goes low when undriven (tristate)\nDetect key press when KEY_Cx goes low during high-to-low strobe of KEY_Rx\nFan originally provided +5V supply the interface but +3.3V works fine"
+	(text "Compatible with original equipment\n\nKey matrix\n- R1+GND: Close lid\n- R2+GND: Open lid\n- R1+C1: Fan off\n- R1+C2: Fan speed up\n- R1+C3: Fan speed down\n- R1+C2+C3: Open / close lid\n- R1+C4: Toggle rain sensor (only certain models)\n- R2+C1: Fan on and cycle speeds\n- R2+C2: Fan on / off\n- R2+C3: Fan intake / exhaust direction\n- R2+C4: Toggle auto thermostat\n\nLEDs\n- LED_AUTO: Auto LED cathode, green with 2.4 V voltage drop\n- LED_RAIN: Rain LED cathode, red with 2 V voltage drop (only certain models)\n\nKEY_Rx and KEY_Cx inputs need pull-ups\nDetect key press when KEY_Rx goes low when undriven (tristate)\nDetect key press when KEY_Cx goes low during high-to-low strobe of KEY_Rx\nFan originally provided +5V supply the interface but +3.3V works fine"
 		(exclude_from_sim no)
 		(at 95.25 59.69 0)
@@
 			)
 		)
+		(property "Alternative" "0022284081"
+			(at 120.65 124.46 0)
+			(effects
+				(font
+					(size 1.27 1.27)
+				)
+				(hide yes)
+			)
+		)
 		(property "LCSC" "C3345591"
 			(at 120.65 124.46 0)
 			(effects
+				(font
+					(size 1.27 1.27)
+				)
+				(hide yes)
+			)
+		)
+		(property "LCSC_Alternative" "C3339252"
+			(at 120.65 124.46 0)
+			(effects
