File: hardware/minuet/v3/lid.kicad_sch (KiCad schematic)
At the start: 11 parts, among them J401 B2B-XH-A, U401 DRV8876PWP

Commit message: First draft of Minuet v3.
Parts:
- added C23: 10n, Capacitor_SMD:C_0603_1608Metric, symbol Device:C
- J9: renamed from J401; Label COVER MOTOR -> LID MOTOR
- R25: renamed from R402; value 2.80K -> 2.21K; footprint Resistor_SMD:R_0603_1608Metric_Pad0.98x0.95mm_HandSolder -> Resistor_SMD:R_0603_1608Metric
- RV1: renamed from RV401; Label COVER CURRENT LIMIT -> CURRENT LIMIT
- renumbered C401 to C19, C402 to C20, C403 to C21, C404 to C22, NT401 to NT4, R401 to R24, TP401 to TP3, U401 to U6
Connections:
- net GND: now also C23.2
- net IPROPI: now also C23.1
Other:
- note added: "LID MOTOR DRIVER"
- note added: "Set overcurrent protection trip current Itrip (A) = 1000 * Vref (V) / Ripropi (Ω) Given Vref = 3.3 V, Ripropi = 2.21 K, Itrip = 1.5 A Must be set high enough to allow the motor to overcome the torque demands of the lid mechanism and ideally should be low enough to detect stall at end of travel. Add a capacitor if there are glitches."
- note removed: "COVER MOTOR DRIVER"
- note removed: "Set overcurrent protection trip current Itrip (A) = 1000 * Vref (V) / Ripropi (Ω) Given Vref = 3.3 V, Ripropi = 2.8 K, Itrip = 1.18 A Must be set high enough to allow the motor to overcome the torque demands of the cover mechanism and low enough to reliably detect stall at end of travel."
- title: Minuet Cover Motor Driver -> Minuet Lid Motor Driver
- moved on the sheet: R25, RV1

Commit message: Prepare for fabrication.
Parts:
- added R25: 10K, Resistor_SMD:R_0603_1608Metric, symbol Device:R
- C19: LCSC (none) -> C377773
- C20, C21: LCSC (none) -> C14663
- C22: LCSC (none) -> C21122
- R24: value 62K -> 51K; LCSC (none) -> C23196
- U6: FT Rotation Offset (none) -> 270
- renumbered R25 to R26
Connections:
- net GND: now also R25.1; no longer R24.1
- new net: R24.1, R25.2
Other:
- note added: "Make 62 K from JLCPCB basic parts"

Commit message: Remove unnecessary fields.
Parts:
- U6: MANUFACTURER Texas Instruments -> (none); MAXIMUM_PACKAGE_HEIGHT 1.2mm -> (none); PACKAGE HTSSOP-16 Texas Instruments -> (none); PARTREV E -> (none); STANDARD Manufacturer Recommendations -> (none)

Commit message: Prepare Minuet v3 for production.
Parts:
- C19, C20, C22: Rating 25V, X5R -> 50V, X5R
- C21: Rating 16V, X5R -> 50V, X5R
- C23: LCSC (none) -> C57112; Rating 6.3V, X5R -> 50V, X5R; now fitted; now in the parts list
- J9: FT Rotation Offset (none) -> 180
Other:
- moved on the sheet: C19, C20, NT4
