File: hardware/minuet/v3/minuet.kicad_pcb (KiCad board)
At the start: 2 copper layers, 79 x 79 mm, 95 parts, among them J101 B2P-VH-B, J102 B2B-XH-A, J103 PPPC062LFBN-RC, J104 B2B-XH-A, J201 USB4105-GF-A, J202 SM04B-SRSS-TB, J301 B3P-VH-B, J302 B5B-XH-A, J401 B2B-XH-A, J501 G800LE300018YEU, J502 MTJ-889X1, J503 MTJ-669X1, Q101 MMBT3904, SW201 EVQ-P7J01P, SW202 EVQ-P7J01P, U101 TSOP39238, U102 LMV331IDCK, U201 TCA9555RTW, U202 ESP32-C3-WROOM-02-N4, U301 MCT8316Z0T, U401 DRV8876PWP

Commit message: First draft of Minuet v3.
Parts:
- removed C304: 22u, Capacitor_SMD:C_0805_2012Metric
- removed C306: 100n, Capacitor_SMD:C_0603_1608Metric
- removed J302: B5B-XH-A, Connector_JST:JST_XH_B5B-XH-A_1x05_P2.50mm_Vertical
- removed L301: 22u, Inductor_SMD:L_0603_1608Metric
- removed NT103: NetTie_2, Generic:NetTie-2_SMD_Pad0.4mm
- removed R301, R303: 18.2K, Resistor_SMD:R_0603_1608Metric
- removed R302: 3.65K, Resistor_SMD:R_0603_1608Metric_Pad0.98x0.95mm_HandSolder
- removed R304, R305, R306: 4.7K, Resistor_SMD:R_0603_1608Metric
- removed R307, R309, R310, R311, R312: 0R, Resistor_SMD:R_0603_1608Metric_Pad0.98x0.95mm_HandSolder
- removed R308: 22K, Resistor_SMD:R_0603_1608Metric_Pad0.98x0.95mm_HandSolder
- removed RN201: 746X101103JP, 746X:RESCAXS64P320X160X70-10N
- removed RV301: 5K, 3362P-1-502LF:TRIM_3362P-1-502LF
- removed TP301: TestPoint_2Pole, TestPoint:TestPoint_2Pads_Pitch2.54mm_Drill0.8mm
- added C18: 1u, Capacitor_SMD:C_0603_1608Metric, F.Cu at (94.8, 60.7)
- added C23: 10n, Capacitor_SMD:C_0603_1608Metric, F.Cu at (104.1, 80.1)
- added J5: B2B-XH-A, Connector_JST:JST_XH_B2B-XH-A_1x02_P2.50mm_Vertical, B.Cu at (99.8, 36.0)
- added NT3: NetTie_2, Generic:NetTie-2_SMD_Pad0.2mm, F.Cu at (61.5, 88.4)
- added R17: 10K, Resistor_SMD:R_0603_1608Metric, F.Cu at (50.0, 94.8)
- added R19: 10K, Resistor_SMD:R_0603_1608Metric, F.Cu at (39.8, 90.5)
- added R21: 10K, Resistor_SMD:R_0603_1608Metric, F.Cu at (82.2, 88.5)
- added R22: 10K, Resistor_SMD:R_0603_1608Metric, F.Cu at (38.5, 91.8)
- added R23: 10K, Resistor_SMD:R_0603_1608Metric, F.Cu at (37.2, 93.0)
- J2: renamed from J102; moved to F.Cu
- J4: renamed from J103; value PPPC062LFBN-RC -> PPPC082LFBN-RC; footprint Connector_PinSocket_2.54mm:PinSocket_2x06_P2.54mm_Vertical -> Connector_PinSocket_2.54mm:PinSocket_2x08_P2.54mm_Vertical
- JP1: renamed from JP101; value SolderJumper_3_Bridged12 -> SolderJumper_2_Bridged; footprint Jumper:SolderJumper-3_P1.3mm_Bridged12_RoundedPad1.0x1.5mm -> Jumper:SolderJumper-2_P1.3mm_Bridged_RoundedPad1.0x1.5mm
- R25: renamed from R402; value 2.80K -> 2.21K; footprint Resistor_SMD:R_0603_1608Metric_Pad0.98x0.95mm_HandSolder -> Resistor_SMD:R_0603_1608Metric
- U5: renamed from U301; value MCT8316Z0T -> MCF8316D; footprint MCT8316Z:MCT8316ZT -> MCF8316D:MCF8316D
- moved C1 26.8 mm to (107.5, 39.2), turned to 90 degrees
- moved J2 17.9 mm to (101.3, 91.3), turned to 180 degrees
- moved C6 16.0 mm to (77.2, 53.5), turned to -45 degrees
- moved R5 14.5 mm to (78.5, 52.2), turned to 135 degrees
- moved C16 13.7 mm to (97.4, 60.7)
- moved R2 13.0 mm to (79.8, 51.0), turned to -45 degrees
- moved J8 12.2 mm to (107.7, 60.0)
- moved C13 11.8 mm to (103.2, 60.8)
- moved C14 11.8 mm to (101.1, 60.8)
- moved U5 11.8 mm to (98.0, 55.8)
- moved C15 11.6 mm to (98.2, 63.8)
- moved C17 11.5 mm to (98.9, 51.5), turned to 0 degrees
- moved R25 11.2 mm to (105.9, 80.1)
- moved NT4 10.8 mm to (104.8, 64.2)
- moved C19 10.3 mm to (105.7, 66.8)
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- renumbered BZ101 to BZ1, C101 to C1, C203 to C10, C204 to C11, C205 to C12, C301 to C13, C302 to C14, C303 to C15, C305 to C16, C307 to C17, C401 to C19, C102 to C2, C402 to C20, C403 to C21, C404 to C22, C103 to C3, C104 to C4, C105 to C5, C106 to C6, C107 to C7, C201 to C8, C202 to C9, D101 to D1, D201 to D2, F101 to F1, J101 to J1, J501 to J10, J502 to J11, J503 to J12, J104 to J3, J201 to J6, J202 to J7, J301 to J8, J401 to J9, L101 to L1, NT101 to NT1, NT102 to NT2, NT401 to NT4, Q101 to Q1, R101 to R1, R110 to R10, R113 to R11, R111 to R12, R112 to R13, R114 to R14, R115 to R15, R116 to R16, R201 to R18, R102 to R2, R202 to R20, R401 to R24, R103 to R3, R104 to R4, R105 to R5, R106 to R6, R107 to R7, R108 to R8, R109 to R9, RV401 to RV1, SW201 to SW1, SW202 to SW2, TP101 to TP1, TP102 to TP2, TP401 to TP3, U101 to U1, U102 to U2, U201 to U3, U202 to U4, U401 to U6, VR101 to VR1
Connections:
- net /cover/CPH renamed /lid/CPH
- net /cover/CPL renamed /lid/CPL
- net /cover/IMODE renamed /lid/IMODE
- net /cover/IPROPI renamed /lid/IPROPI
- net /cover/OUT1 renamed /lid/OUT1
- net /cover/OUT2 renamed /lid/OUT2
- net /cover/VCP renamed /lid/VCP
- net /cover/VM renamed /lid/VM
- net /fan/U renamed /fan/A
- net /fan/V renamed /fan/B
- net /fan/W renamed /fan/C
- net Net-(VR101-EN) renamed /VIN
- C17 pad 1: /fan/AVDD -> Net-(U5-AVDD)
- J4 pad 10: +3.3V -> UART_TXD
- J4 pad 11: GND -> unconnected-(J4-Pin_11-Pad11)
- J4 pad 12: +12V -> LOCK
- J4 pad 5: SDA -> GPIO6
- J4 pad 6: SCL -> GPIO5
- J4 pad 7: UART_RXD -> SCL
- J4 pad 8: UART_TXD -> SDA
- J4 pad 9: GND -> UART_RXD
- R1 pad 2: XIO15 -> XIO14
- R8 pad 2: XIO14 -> XIO13
- U4 pad 5: SCL -> GPIO6
- U4 pad 7: GPIO8_STRAP -> SCL
- U5 pad 1: unconnected-(U301-NC-Pad1) -> Net-(U5-DVDD)
- U5 pad 22: XIO13 -> GND
- U5 pad 23: XIO14 -> GND
- U5 pad 24: unconnected-(U301-VSEL_BK-Pad24) -> GND
- U5 pad 25: /fan/AVDD -> GND
- U5 pad 27: /fan/U_HALL -> Net-(U5-AVDD)
- U5 pad 28: unconnected-(U301-HNA-Pad28) -> XIO13
- U5 pad 29: /fan/V_HALL -> unconnected-(U5-FG-Pad29)
- U5 pad 3: /fan/VBK -> +3.3V
- U5 pad 30: unconnected-(U301-HNB-Pad30) -> SDA
- U5 pad 31: /fan/W_HALL -> SCL
- U5 pad 32: unconnected-(U301-HNC-Pad32) -> GND
- U5 pad 33: /fan/MODE -> GND
- U5 pad 34: /fan/SLEW -> GND
- U5 pad 35: /fan/ADVANCE -> GND
- U5 pad 36: XIO12 -> unconnected-(U5-DACOUT1-Pad36)
- U5 pad 37: /fan/ILIM -> unconnected-(U5-DACOUT2-Pad37)
- U5 pad 38: GND -> unconnected-(U5-DACOUT2/SOX-Pad38)
- U5 pad 39: GPIO5 -> unconnected-(U5-ALARM-Pad39)
- U5 pad 40: GPIO8_STRAP -> XIO12
- U5 pad 5: Net-(U301-SW_BK) -> unconnected-(U5-SW_BK-Pad5)
Routing:
- net /fan/AVDD: track 89.8 -> 0.00 mm
- net GPIO8_STRAP: track 71.9 -> 0.00 mm, vias 4 -> 0
- net LOCK: track 0.00 -> 71.6 mm, vias 0 -> 3
- net XIO14: track 70.4 -> 2.99 mm, vias 2 -> 0
- net SDA: track 63.9 -> 117.9 mm, vias 4 -> 3
- net /fan/ILIM: track 48.6 -> 0.00 mm, vias 2 -> 0
- net +3.3V: track 237.8 -> 285.3 mm, vias 8 -> 12
- net /fan/VBK: track 46.5 -> 0.00 mm, vias 4 -> 0
- net SCL: track 69.1 -> 112.2 mm, vias 4 -> 3
- net /fan/MODE: track 34.1 -> 0.00 mm
- net GPIO6: track 0.00 -> 33.9 mm
- net /fan/SLEW: track 32.1 -> 0.00 mm
- net Net-(JP101-B): track 30.0 -> 0.00 mm
- net GPIO5: track 65.1 -> 36.4 mm, vias 4 -> 0
- net GPIO3: track 62.5 -> 35.6 mm
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Other:
- board text added: "12V 3V3 LOCK TXD SDA GPIO5 GPIO0 RESET"
- board text added: "GND GND (NC) RXD SCL GPIO6 GPIO1 BOOT"
- board text added: "LID MOTOR"
- board text added: "LID MOTOR CURRENT LIMIT"
- board text added: "LOCK"
- board text added: "SOUND"
- board text added: "github.com/j9brown/minuet Brown Studios Minuet Fan Controller 2025/5, v3.0"
- board text removed: "+ADV-"
- board text removed: "+MODE-"
- board text removed: "+SLEW-"
- board text removed: "12V 3V3 TXD SCL GPIO0 RESET"
- board text removed: "COVER CURRENT LIMIT"
- board text removed: "COVER MOTOR"
- board text removed: "FAN CURRENT LIMIT"
- board text removed: "FAN SENSOR"
- board text removed: "GND GND RXD SDA GPIO1 BOOT"
- board text removed: "ILIM"
- board text removed: "VOLUME"
- board text removed: "github.com/j9brown/minuet Brown Studios Minuet Fan Controller 2025/2, v2.1"

Commit message: Prepare for fabrication.
Parts:
- added R25: 10K, Resistor_SMD:R_0603_1608Metric, F.Cu at (109.5, 76.8)
- R14: value 1.5M -> 1M
- R24: value 62K -> 51K
- R9: value 100K -> 68K
- SW1, SW2: value EVQ-P7J01P -> EVQ-P7A01P
- moved C7 22.8 mm to (83.8, 109.0), turned to 0 degrees
- moved R12 12.6 mm to (106.5, 97.0), turned to -90 degrees
- moved R13 9.76 mm to (109.0, 97.0), turned to -90 degrees
- moved R24 3.25 mm to (106.0, 76.8)
- moved R10 1.35 mm to (83.8, 106.5), turned to 180 degrees
- moved C1 0.79 mm to (107.2, 40.0)
- moved C23 0.50 mm to (104.2, 80.6)
- moved R26 0.50 mm to (106.0, 80.6)
- moved RV1 0.50 mm to (108.0, 81.5)
- moved TP3 0.50 mm to (102.0, 82.8)
- renumbered R25 to R26
Connections:
- R24 pad 1: GND -> Net-(R24-Pad1)
Routing:
- net Net-(J3-Pin_2): track 20.9 -> 7.46 mm
- net Net-(J3-Pin_1): track 15.0 -> 3.92 mm
- net /RSEN: track 37.2 -> 46.2 mm
- net /lid/IMODE: track 8.97 -> 5.13 mm
- net Net-(R24-Pad1): track 0.00 -> 1.85 mm
- net +3.3V: track 285.3 -> 283.8 mm
- net GND: track 96.5 -> 97.6 mm
- net +12V: track 70.8 -> 70.2 mm
- net /lid/IPROPI: track 10.6 -> 11.1 mm

Commit message: Prepare Minuet v3 for production.
Parts:
- added TH1: JLCPCB_PCBA_Tooling_Hole, Generic:JLCPCB_PCBA_Tooling_Hole, F.Cu at (110.0, 45.0)
- added TH2: JLCPCB_PCBA_Tooling_Hole, Generic:JLCPCB_PCBA_Tooling_Hole, F.Cu at (110.0, 110.0)
- added TH3: JLCPCB_PCBA_Tooling_Hole, Generic:JLCPCB_PCBA_Tooling_Hole, F.Cu at (35.0, 94.8)
- C1, F1: moved to F.Cu
- SW1, SW2: footprint EVQ-P7A01P:SW_EVQ-P7A01P -> Button_Switch_SMD:SW_SPST_EVQP7A
- moved R26 0.95 mm to (106.2, 81.5)
- moved C23 0.90 mm to (104.2, 81.5)
- renumbered R9 to R10, R12 to R11, R11 to R12, R10 to R9
Routing:
- net /12V_IN: track 6.23 -> 5.03 mm
- net /lid/IPROPI: track 11.1 -> 10.5 mm
Other:
- board text added: "${COMPANY} ${TITLE} ${ISSUE_DATE}, ${REVISION} ${COMMENT1}"
- board text removed: "github.com/j9brown/minuet Brown Studios Minuet Fan Controller 2025/5, v3.0"
